File: eagle_pcb_files/main_board/main.brd (EAGLE design)
At the start: 73.6 x 34.3 mm, 20 parts

Commit message: Temporary version of main board
:')
Parts:
- removed FRAME2: FRAME-LEDGER, SparkFun-Aesthetics:CREATIVE_COMMONS
- added C1, C2, C3, C4, C5, C6, C7: (no value), rcl:C0402
- added U$3, U$9: POLOLU_FUEL_GAUGEBREAKBOARD, SparFun-FuelGauge:BREAKBOARD
- moved U$5 5.12 mm to (9.40, 13.1)
- moved RAO1 4.70 mm to (34.4, 15.4)
- moved RAO3 4.26 mm to (7.49, 14.4), turned to 0 degrees
- moved BAT1 3.94 mm to (6.22, 0.64)
- moved FUSE1 3.94 mm to (12.6, 0.64)
- moved RAO4 3.84 mm to (61.2, 14.2), turned to 0 degrees
- moved D1 3.81 mm to (7.49, 5.21)
- moved FUSE2 2.80 mm to (56.8, 0.76)
- moved BAT2 2.67 mm to (65.0, 0.89)
- moved R1 1.55 mm to (38.1, 5.97)
- moved U$2 1.27 mm to (72.6, 16.3)
- moved U$1 0.64 mm to (24.1, -0.25)
Connections:
- net 3.3V: now also C1.2, C2.1, C3.1, C4.1, C5.2, C6.1, C7.1, U$3.VCC, U$9.VCC
- net B2: now also RAO2.31
- net GND: now also C1.1, C2.2, C3.2, C4.2, C5.1, C6.2, C7.2, U$3.-, U$3.GND, U$9.-, U$9.GND
- net SCL: now also U$3.SCL, U$9.SCL
- net SDA: now also U$3.SDA, U$9.SDA
- net VIN1: now also U$3.+
- net VIN2: now also U$9.+
Routing:
- net G1: track 96.1 -> 0.00 mm
- net 3.3V: track 73.7 -> 0.00 mm, vias 4 -> 0
- net SS2: track 69.7 -> 0.00 mm
- net SCL: track 64.4 -> 0.00 mm, vias 6 -> 0
- net MOSI: track 61.1 -> 0.00 mm, vias 3 -> 0
- net SDA: track 60.2 -> 0.00 mm, vias 6 -> 0
- net G2: track 57.7 -> 0.00 mm, vias 1 -> 0
- net SCK: track 53.7 -> 0.00 mm, vias 4 -> 0
- net NSS: track 47.0 -> 0.00 mm, vias 4 -> 0
- net MISO: track 44.9 -> 0.00 mm, vias 5 -> 0
- net G3: track 34.9 -> 0.00 mm
- net DIO0: track 29.3 -> 0.00 mm
- net DIO2: track 29.3 -> 0.00 mm, vias 1 -> 0
- net DIO3: track 25.7 -> 0.00 mm, vias 2 -> 0
- net DIO1: track 25.4 -> 0.00 mm, vias 1 -> 0
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